File: PCB/final_project3.brd (EAGLE design)
At the start: 74.9 x 52.1 mm, 19 parts

Commit message: Correction
Connections:
- net GND3: now also REGULATOR.2
Routing:
- net GND3: track 128.3 -> 177.1 mm
Changed lines of the file:
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@@
 <wire x1="5.08" y1="49.53" x2="5.08" y2="27.94" width="1" layer="1"/>
 <wire x1="5.08" y1="49.53" x2="58.42" y2="49.53" width="1" layer="1"/>
+<contactref element="REGULATOR" pad="2"/>
+<wire x1="71.12" y1="17.78" x2="73.3124" y2="17.78" width="1" layer="1"/>
+<wire x1="73.3124" y1="17.78" x2="73.3124" y2="49.53" width="1" layer="1"/>
+<wire x1="73.3124" y1="49.53" x2="58.42" y2="49.53" width="1" layer="1"/>
 </signal>
 <signal name="N$2">

Commit message: Final
Parts:
- removed J6, J8, J9: (no value), SparkFun-Connectors:1X01
- added J1, J3, J4: (no value), SparkFun-Connectors:1X01
- J5: device SparkFun-Connectors:1X01 -> SparkFun-Connectors:1X02
- moved J5 51.1 mm to (82.5, 19.1), turned to 270 degrees
- moved J11 15.3 mm to (12.7, 45.7)
- moved J10 15.3 mm to (15.2, 45.7)
- moved J2 5.24 mm to (20.3, 30.5)
- moved LED 4.02 mm to (66.0, 41.9)
- moved BUTTON 4.02 mm to (52.1, 41.9)
- moved R1 4.02 mm to (68.6, 34.3)
- moved R2 4.02 mm to (49.5, 34.3)
- moved PSOC[VDD-GND] 4.02 mm to (67.3, 6.35)
- moved PSOC[P_2.1-P_2.7] 4.02 mm to (67.3, 26.7)
- moved REGULATOR 4.02 mm to (74.9, 19.1)
- moved PSOC[P_1.6-P_1.7-GND] 4.02 mm to (14.0, 26.7)
- moved PSOC[P_3.3-GND] 4.02 mm to (6.35, 6.35)
- moved PSOC_FIVEPINS 4.02 mm to (6.35, 11.4)
- moved PSOC[P_12.0-P_12.1] 4.02 mm to (31.8, 26.7)
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Connections:
- new net N$1: J5.1, REGULATOR.1
- net GND3: now also J3.1, J4.1, J5.2, R1.P$1, R2.P$1; no longer J5.1
- net VDD: now also J1.1; no longer J6.1, R1.P$1, R2.P$1
Routing:
- net VDD: track 216.9 -> 149.6 mm
- net N$2: track 19.0 -> 7.93 mm
- net N$3: track 16.5 -> 26.9 mm
- net N$4: track 16.5 -> 26.9 mm
- net N$1: track 0.00 -> 7.62 mm
- net GND3: track 177.1 -> 170.6 mm
- net LED: track 16.0 -> 15.3 mm
- added copper zone on layer 1, net GND3
Other:
- board size 74.9 x 52.1 mm -> 86.4 x 50.8 mm
